File: DragonBoard-sub-board-backup.sch (EAGLE design)
At the start: 15 parts, among them U1 TXB0108PWR, U2 TXB0108PWR, U3 62674-301121ALF, U4 62674-301121ALF

Commit message: added ftdi chip
Parts:
- added .1UF, .1UF1, .1UF2, .1UF3, .1UF4, 4.7UF, 4.7UF1, 4.7UF2, 4.7UF3, 4.7UF4, 4.7UF5, C1, C10, C11, C12, C13, C14, C15, C16, C17, C18, C19, C2, C20, C21, C22, C23, C24, C25, C26, C27, C28, C29, C3, C30, C4, C5, C6, C7, C8, C9: (no value), rcl:C-USC0402
- added IC1: REG1117, burr-brown:REG1117
- added IC2: 93AA76A, microchip:93AA76A
- added JP2: (no value), pinhead:PINHD-2X3
- added JP3: (no value), pinhead:PINHD-1X3
- added JP4, JP6: (no value), pinhead:PINHD-1X6
- added JP5: (no value), pinhead:PINHD-2X2
- added JP7, JP8, JP9: (no value), pinhead:PINHD-1X4
- added L1, L2: (no value), rcl:L-USL3216C
- added Q2: 8MHz, crystal:CRYSTALCTS406
- added R1, R2, R3, R4, R5: (no value), rcl:R-US_R0402
- added U$4: FT423H, FT432H:FT423H
- added U5: NC7ST04M5X, pca9685:NC7ST04M5X
Connections:
- removed net !CS: J3.3
- removed net AD0/SDO: J3.2
- removed net FSYNC: J2.2
- removed net I2C_SDA: U$1LS.21
- removed net N$13: U1.B8, U2.B8
- removed net N$15: U1.B6, U2.B6
- removed net N$16: U1.B5, U2.B5
- removed net N$18: U1.B3, U2.B3
- removed net N$19: U1.B2, U2.B2
- removed net N$20: U1.B1, U2.B1
- removed net SCL: JP1.4
- removed net SCL/SCLK: J1.1
- removed net SDA: JP1.5
- removed net SDA/SDI: J1.2
- removed net SPI1_CS_N: U2.A7
- removed net VDD: J1.3, JP1.2
- new net 3.3V: IC2.VCC
- new net CAM_SCL: U$1HS.32, U3.13, U4.13
- new net CAM_SDA: U$1HS.34, U3.14, U4.14
- new net CON_RX: JP6.4, U1.B5
- new net CON_TX: JP6.5, U1.B6
- new net CSI0_C+: U$1HS.2, U3.3
- new net CSI0_C-: U$1HS.4, U3.2
- new net CSI0_D0+: U$1HS.8, U3.9
- new net CSI0_D0-: U$1HS.10, U3.8
- new net CSI0_D1+: U$1HS.14, U3.6
- new net CSI0_D1-: U$1HS.16, U3.5
- new net CSI0_D2+: U$1HS.20, U3.25
- new net CSI0_D2-: U$1HS.22, U3.26
- new net CSI0_D3+: U$1HS.26, U3.28
- new net CSI0_D3-: U$1HS.28, U3.29
- new net CSI1_C+: U$1HS.54, U4.3
- new net CSI1_C-: U$1HS.56, U4.2
- new net CSI1_D0+: U$1HS.42, U4.9
- new net CSI1_D0-: U$1HS.44, U4.8
- new net CSI1_D1+: U$1HS.48, U4.6
- new net CSI1_D1-: U$1HS.50, U4.5
- new net DSI_CLK+: U$1HS.21
- new net DSI_CLK-: U$1HS.23
- new net DSI_D0+: U$1HS.27
- new net DSI_D0-: U$1HS.29
- new net DSI_D1+: U$1HS.33
- new net DSI_D1-: U$1HS.35
- new net DSI_D2+: U$1HS.39
- new net DSI_D2-: U$1HS.41
- new net DSI_D3+: U$1HS.45
- new net DSI_D3-: U$1HS.47
- new net EECLK: IC2.CLK, U$4.EECLK
- new net EECS: IC2.CS, U$4.EECS
- new net EEDATA: IC2.DI, R5.2, U$4.EEDATA
- new net GPS_RX: U1.B7
- new net GPS_TX: U1.B8
- new net HSIC_DATA: U$1HS.59
- new net HSIC_STR: U$1HS.57
- new net I2C1_SDA: JP1.5, JP2.1, JP5.4, U$1LS.21
- new net I2C3_SCL: U$1HS.36
- new net I2C3_SDA: U$1HS.38
- new net MCLK0: U$1HS.15, U3.11
- new net MCLK1: U$1HS.17, U4.11
- new net N$1: JP3.2, U$2.PS
- new net N$10: U$3.ECL
- new net N$11: C25.1, Q2.2, R3.2, U$4.OSCO
- new net N$12: U$3.INT
- new net N$2: JP2.3, U$2.SDA
- new net N$3: JP2.4, U$2.SCL
- new net N$4: JP4.4, JP5.1
- new net N$5: JP4.3, JP5.3
- new net N$6: C30.1, R4.2, U$4.REF
- new net N$7: C26.1, Q2.1, R3.1, U$4.OSIC
- new net N$8: U$3.ECA
- new net SBUS: JP8.2, U5.A
- new net SPI1_CS: U$1HS.7, U2.A7
- new net SPI_A_CLK: J1.1, U$3.SCL, U1.B4
- new net SPI_A_CS: J3.3, U$3.NCS, U1.B2
- new net SPI_A_MISO: J1.2, U$3.AD0, U1.B3
- new net SPI_A_MOSI: J3.2, U$3.SDA, U1.B1
- new net SPI_B_CLK: JP2.6, U2.B5
- new net SPI_B_CS: U$2.CSB, U2.B7
- new net SPI_B_MISO: U$2.SDO, U2.B6
- new net SPI_B_MOSI: JP2.5, U2.B8
- new net USB_D+: JP9.3, U$1HS.51, U$4.DP
- new net USB_D-: JP9.2, U$1HS.53, U$4.DM
- new net VCORE: .1UF3.1, 4.7UF3.1, C28.1, C29.1, U$4.VCORE1, U$4.VCORE2, U$4.VREGOUT
- new net VPHY: .1UF2.1, 4.7UF2.1, L2.2, U$4.VPHY
- new net VPLL: .1UF1.1, 4.7UF1.1, L1.2, U$4.VPLL
- new net _SBUS: JP8.1, U5.Y
- net +1.8V: now also C14.1, C15.1, C22.1, C23.1, C3.1, C5.1, U3.21, U4.21
- net +3.3V: now also .1UF.1, .1UF4.1, 4.7UF.1, 4.7UF4.1, 4.7UF5.1, C1.1, C12.1, C13.1, C2.1, C20.1, C21.1, C27.1, C4.1, C7.1, IC1.VOUT, J1.3, JP1.2, JP3.1, JP4.2, JP4.5, JP7.4, L1.1, L2.1, U$2.VCC, U$3.VCC, U$4.VCCIO1, U$4.VCCIO2, U$4.VCCIO3, U$4.VREGIN, U3.12, U4.12, U5.VCC
- net +5V: now also C10.1, C11.1, C18.1, C19.1, C24.1, C6.1, IC1.VIN, JP4.1, JP8.3, JP9.1, R1.2, U3.17, U4.17
- net FLASH: now also U3.19, U4.19
- net GND: now also .1UF.2, .1UF1.2, .1UF2.2, .1UF3.2, .1UF4.2, 4.7UF.2, 4.7UF1.2, 4.7UF2.2, 4.7UF3.2, 4.7UF4.2, 4.7UF5.2, C1.2, C10.2, C11.2, C12.2, C13.2, C14.2, C15.2, C16.2, C17.2, C18.2, C19.2, C2.2, C20.2, C21.2, C22.2, C23.2, C24.2, C25.2, C26.2, C27.2, C28.2, C29.2, C3.2, C30.2, C4.2, C5.2, C6.2, C7.2, C8.2, C9.2, IC1.GND, IC2.GND, J2.2, JP3.3, JP4.6, JP6.1, JP7.3, JP8.4, JP9.4, R2.1, R4.1, U$2.GND, U$3.FSYNC, U$3.GND, U$4.GND1, U$4.GND2, U$4.GND3, U$4.TEST, U2.GND, U3.1, U3.10, U3.16, U3.18, U3.23, U3.24, U3.27, U3.30, U3.4, U3.7, U4.1, U4.10, U4.16, U4.18, U4.23, U4.24, U4.27, U4.30, U4.4, U4.7, U5.GND
- net I2C0_SCL: now also JP7.2
- net I2C0_SDA: now also JP7.1
- net I2C1_SCL: now also JP1.4, JP2.2, JP5.2
- net N$14: now also IC2.DO, R5.1; no longer U1.B7, U2.B7
- net N$17: now also R1.1, R2.2, U$4.RESET; no longer U1.B4, U2.B4
- net RESET0: now also U3.20
- net RESET1: now also U4.20
- net SPI0_CLK: now also U1.A4; no longer U1.A5
- net SPI0_CS_N: now also U1.A2; no longer U1.A7
- net SPI0_MISO: now also U1.A3; no longer U1.A6
- net SPI0_MOSI: now also U1.A1; no longer U1.A8
- net SPI1_CLK: now also U$1HS.9
- net SPI1_MISO: now also U$1HS.11
- net SPI1_MOSI: now also U$1HS.1
- net STANDBY0: now also U3.15
- net STANDBY1: now also U4.15
- net SYS_DCIN: now also C16.1, C17.1, C8.1, C9.1, U3.22, U4.22
- net UART0_RX: now also U1.A7; no longer U1.A1
- net UART0_TX: now also U1.A8; no longer U1.A2
- net UART1_RX: now also U1.A5; no longer U1.A4
- net UART1_TX: now also U1.A6; no longer U1.A3
Other:
- note added: "Motherboard MCU Crystal"
- moved on the sheet: U$1ANALOG, U$1HS, U$3, U2, U3, U4
