File: DragonBoard-sub-board-backup.sch (EAGLE design)
At the start: 77 parts, among them IC1 REG1117, IC2 93AA76A, Q2 8MHz, U1 TXB0108PWR, U2 TXB0108PWR, U3 62674-301121ALF, U4 62674-301121ALF, U5 NC7ST04M5X

Commit message: Done with baord
Parts:
- added C31, C32: 0.1uF, rcl:C-USC0805
- added JP11, JP12, JP13: (no value), pinhead:PINHD-1X4
- C1, C10, C100, C102, C104, C106, C107, C108, C109, C11, C110, C12, C13, C14, C15, C16, C17, C18, C19, C20, C21, C22, C23, C24, C28, C30, C4, C5, C8, C9: value (none) -> 0.1uF
- C101, C103, C105, C27, C29: value (none) -> 4.7uF
- C2, C3: value (none) -> 0.1Uf
- C25, C26: value (none) -> 30pF
- C6, C7: value (none) -> 1uF
- L1, L2: value (none) -> 0.1uH
- Q2: value 8MHz -> 12MHz
- R1: value (none) -> 1K
- R2, R3: value (none) -> 100k
- R4: value (none) -> 12k
- R5: value (none) -> 22k
- U$1: value DRAGON-BOARD -> DRAGON-BOARD-TH; device DragonBoard:DRAGON-BOARD -> DragonBoard:DRAGON-BOARD-TH
- renumbered .1UF to C100, .1UF1 to C103, .1UF2 to C105, .1UF3 to C106, .1UF4 to C108, 4.7UF to C101, 4.7UF1 to C102, 4.7UF2 to C104, 4.7UF3 to C107, 4.7UF4 to C109, 4.7UF5 to C110
Connections:
- removed net 3.3V: IC2.VCC
- removed net SBUS_RX: JP8.2, U5.Y
- removed net SBUS_TX: JP8.1
- new net ADBUS_RX: JP8.2, U$4.ADBUS1, U5.Y
- new net ADBUS_TX: JP8.1, U$4.ADBUS0
- new net BDBUS_RX: JP11.2, U$4.BDBUS1
- new net BDBUS_TX: JP11.1, U$4.BDBUS0
- new net CDBUS_RX: JP12.2, U$4.CDBUS1
- new net CDBUS_TX: JP12.1, U$4.CDBUS0
- new net DDBUS_RX: JP13.2, U$4.DDBUS1
- new net DDBUS_TX: JP13.1, U$4.DDBUS0
- net +3.3V: now also C31.1, C32.1, IC2.VCC, JP11.3, JP12.3, JP13.3
- net CDC_HPH_L: now also U$1A.10; no longer U$1ANALOG.10
- net CDC_HPH_R: now also U$1A.8; no longer U$1ANALOG.8
- net CDC_HPH_REF: now also U$1A.9; no longer U$1ANALOG.9
- net CDC_HS_DET: now also U$1A.11; no longer U$1ANALOG.11
- net CDC_MIC2_P: now also U$1A.6; no longer U$1ANALOG.6
- net CDC_MIC3_P: now also U$1A.7; no longer U$1ANALOG.7
- net CDC_MIC_BIAS1: now also U$1A.12; no longer U$1ANALOG.12
- net GND: now also C31.2, C32.2, JP11.4, JP12.4, JP13.4, U$1A.4; no longer U$1ANALOG.4
- net GND_CFILT: now also U$1A.5; no longer U$1ANALOG.5
- net N$9: now also U$1A.15; no longer U$1ANALOG.15
- net SPKR_OUT_M: now also U$1A.2; no longer U$1ANALOG.2
- net SPKR_OUT_P: now also U$1A.1; no longer U$1ANALOG.1
- net VPH_PWR: now also U$1A.3; no longer U$1ANALOG.3

Commit message: Fixed missing traces and some values. Also added bmp logos.
Parts:
- removed C108, C109, C110: 0.1uF, rcl:C-USC0402
- removed IC2: 93AA76A, microchip:93AA76A
- removed JP13: (no value), pinhead:PINHD-1X4
- added C33, C35: 0.1uF, rcl:C-USC0402
- added C34: 4.7uF, rcl:C-USC0402
- added IC100: REG1117, burr-brown:REG1117
- added JP100: (no value), pinhead:PINHD-2X2
- C101, C103, C27, C29: value 4.7uF -> 0.1uF
- C105: value 4.7uF -> 1uF
- C106: value 0.1uF -> 1uF
- C11, C12: value 0.1uF -> 30pF
- C14, C17, C19: value 0.1uF -> 4.7uF
- C18, C23: value 0.1uF -> 0.1Uf
- C2, C3: value 0.1Uf -> 0.1uF
- C21: value 0.1uF -> NC
- C25: value 30pF -> 4.7uF
- C26: value 30pF -> 0.1uF
- C31, C32: device rcl:C-USC0805 -> rcl:C-USC0402
- C6, C7: value 1uF -> 0.1uF
- C8, C9: device rcl:C-USC0402 -> rcl:C-USC0805
- IC1: value REG1117 -> 93AA76A; device burr-brown:REG1117 -> microchip:93AA76A
- JP1: device mike-temp:M05_ROUNDONLY_NOSILK -> pinhead:PINHD-1X6
- JP11: device pinhead:PINHD-1X4 -> pinhead:PINHD-1X5
- JP12: device pinhead:PINHD-1X4 -> pinhead:PINHD-1X6
- JP2: device pinhead:PINHD-2X3 -> pinhead:PINHD-1X4
- JP3: device pinhead:PINHD-1X3 -> mike-temp:M05_ROUNDONLY_NOSILK
- JP4: device pinhead:PINHD-1X6 -> pinhead:PINHD-2X3
- JP5: device pinhead:PINHD-2X2 -> pinhead:PINHD-1X3
- JP6: device pinhead:PINHD-1X6 -> pinhead:PINHD-1X4
- JP8: device pinhead:PINHD-1X5 -> pinhead:PINHD-1X4
- R1: value 1K -> NC
- R2: value 100k -> 2k
- R3: value 100k -> 12k
- R4: value 12k -> 10k
- R5: value 22k -> 15K
- U$1: value DRAGON-BOARD-TH -> GY-63; device DragonBoard:DRAGON-BOARD-TH -> imu:GY-63
- U$2: value GY-63 -> GY-9250; device imu:GY-63 -> imu:GY-9250
- U$3: value GY-9250 -> FT423H; device imu:GY-9250 -> FT432H:FT423H
- U$4: value FT423H -> DRAGON-BOARD-TH; device FT432H:FT423H -> DragonBoard:DRAGON-BOARD-TH
- renumbered Q2 to Q1
Connections:
- net +1.8V: now also C101.1, C107.1, C32.1, C4.1, U$4LS.35; no longer C14.1, C15.1, C22.1, C3.1, U$1LS.35
- net +3.3V: now also C10.1, C103.1, C104.1, C105.1, C14.1, C18.1, C22.1, C30.1, C34.1, C35.1, C6.1, C8.1, C9.1, IC1.VCC, IC100.VOUT, JP1.5, JP2.4, JP3.2, JP5.1, JP6.3, JP8.3, JP9.3, U$1.VCC, U$3.VCCIO, U$3.VREGIN; no longer C1.1, C100.1, C101.1, C108.1, C109.1, C110.1, C12.1, C20.1, C21.1, C27.1, C32.1, C4.1, C7.1, IC1.VOUT, IC2.VCC, JP11.3, JP12.3, JP13.3, JP3.1, JP4.2, JP4.5, JP7.4, U$3.VCC, U$4.VCCIO, U$4.VREGIN
- net +5V: now also C102.1, C106.1, C16.1, C28.1, C29.1, C3.1, IC100.VIN, JP1.1, JP11.4, JP7.1, R5.2, U$4LS.37; no longer C10.1, C11.1, C18.1, C19.1, C24.1, C6.1, IC1.VIN, JP4.1, JP8.4, JP9.1, R1.2, U$1LS.37
- net ADBUS_RX: now also JP11.2, U$3.ADBUS1; no longer JP8.2, U$4.ADBUS1
- net ADBUS_TX: now also JP11.1, U$3.ADBUS0; no longer JP8.1, U$4.ADBUS0
- net BDBUS_RX: now also JP9.2, U$3.BDBUS1; no longer JP11.2, U$4.BDBUS1
- net BDBUS_TX: now also JP9.1, U$3.BDBUS0; no longer JP11.1, U$4.BDBUS0
- net CAM_SCL: now also U$4HS.32; no longer U$1HS.32
- net CAM_SDA: now also U$4HS.34; no longer U$1HS.34
- net CDBUS_RX: now also JP8.2, U$3.CDBUS1; no longer JP12.2, U$4.CDBUS1
- net CDBUS_TX: now also JP8.1, U$3.CDBUS0; no longer JP12.1, U$4.CDBUS0
- net CDC_HPH_L: now also U$4A.10; no longer U$1A.10
- net CDC_HPH_R: now also U$4A.8; no longer U$1A.8
- net CDC_HPH_REF: now also U$4A.9; no longer U$1A.9
- net CDC_HS_DET: now also U$4A.11; no longer U$1A.11
- net CDC_MIC2_P: now also U$4A.6; no longer U$1A.6
- net CDC_MIC3_P: now also U$4A.7; no longer U$1A.7
- net CDC_MIC_BIAS1: now also U$4A.12; no longer U$1A.12
- net CON_RX: now also JP12.4; no longer JP6.4
- net CON_TX: now also JP12.5; no longer JP6.5
- net CSI0_C+: now also U$4HS.2; no longer U$1HS.2
- net CSI0_C-: now also U$4HS.4; no longer U$1HS.4
- net CSI0_D0+: now also U$4HS.8; no longer U$1HS.8
- net CSI0_D0-: now also U$4HS.10; no longer U$1HS.10
- net CSI0_D1+: now also U$4HS.14; no longer U$1HS.14
- net CSI0_D1-: now also U$4HS.16; no longer U$1HS.16
- net CSI0_D2+: now also U$4HS.20; no longer U$1HS.20
- net CSI0_D2-: now also U$4HS.22; no longer U$1HS.22
- net CSI0_D3+: now also U$4HS.26; no longer U$1HS.26
- net CSI0_D3-: now also U$4HS.28; no longer U$1HS.28
- net CSI1_C+: now also U$4HS.54; no longer U$1HS.54
- net CSI1_C-: now also U$4HS.56; no longer U$1HS.56
- net CSI1_D0+: now also U$4HS.42; no longer U$1HS.42
- net CSI1_D0-: now also U$4HS.44; no longer U$1HS.44
- net CSI1_D1+: now also U$4HS.48; no longer U$1HS.48
- net CSI1_D1-: now also U$4HS.50; no longer U$1HS.50
- net DDBUS_RX: now also JP6.2, U$3.DDBUS1; no longer JP13.2, U$4.DDBUS1
- net DDBUS_TX: now also JP6.1, U$3.DDBUS0; no longer JP13.1, U$4.DDBUS0
- net DSI_BLCTRL: now also U$4LS.28; no longer U$1LS.28
- net DSI_CLK+: now also U$4HS.21; no longer U$1HS.21
- net DSI_CLK-: now also U$4HS.23; no longer U$1HS.23
- net DSI_D0+: now also U$4HS.27; no longer U$1HS.27
- net DSI_D0-: now also U$4HS.29; no longer U$1HS.29
- net DSI_D1+: now also U$4HS.33; no longer U$1HS.33
- net DSI_D1-: now also U$4HS.35; no longer U$1HS.35
- net DSI_D2+: now also U$4HS.39; no longer U$1HS.39
- net DSI_D2-: now also U$4HS.41; no longer U$1HS.41
- net DSI_D3+: now also U$4HS.45; no longer U$1HS.45
- net DSI_D3-: now also U$4HS.47; no longer U$1HS.47
- net EECLK: now also IC1.CLK, U$3.EECLK; no longer IC2.CLK, U$4.EECLK
- net EECS: now also IC1.CS, U$3.EECS; no longer IC2.CS, U$4.EECS
- net EEDATA: now also IC1.DI, R2.2, U$3.EEDATA; no longer IC2.DI, R5.2, U$4.EEDATA
- net FLASH: now also U$4LS.23; no longer U$1LS.23
- net GND: now also C33.2, C34.2, C35.2, IC100.GND, JP1.6, JP11.5, JP12.1, JP2.3, JP5.3, JP6.4, JP7.4, JP8.4, R3.1, U$1.GND, U$2.FSYNC, U$3.TEST, U$4A.4, U$4HS.12, U$4HS.13, U$4HS.18, U$4HS.19, U$4HS.24, U$4HS.25, U$4HS.30, U$4HS.31, U$4HS.37, U$4HS.43, U$4HS.46, U$4HS.49, U$4HS.52, U$4HS.55, U$4HS.58, U$4HS.6, U$4LS.1, U$4LS.2, U$4LS.39, U$4LS.40; no longer C108.2, C109.2, C110.2, IC2.GND, JP1.3, JP11.4, JP12.4, JP13.4, JP4.6, JP6.1, JP7.3, JP8.5, R2.1, U$1A.4, U$1HS.12, U$1HS.13, U$1HS.18, U$1HS.19, U$1HS.24, U$1HS.25, U$1HS.30, U$1HS.31, U$1HS.37, U$1HS.43, U$1HS.46, U$1HS.49, U$1HS.52, U$1HS.55, U$1HS.58, U$1HS.6, U$1LS.1, U$1LS.2, U$1LS.39, U$1LS.40, U$3.FSYNC, U$4.GND, U$4.TEST
- net GND_CFILT: now also U$4A.5; no longer U$1A.5
- net GPIO_110: now also U$4LS.16; no longer U$1LS.16
- net GPIO_113: now also U$4LS.18; no longer U$1LS.18
- net GPIO_114: now also U$4LS.20; no longer U$1LS.20
- net GPIO_115: now also U$4LS.27; no longer U$1LS.27
- net GPIO_12: now also U$4LS.24; no longer U$1LS.24
- net GPIO_13: now also U$4LS.25; no longer U$1LS.25
- net GPIO_24: now also U$4LS.29; no longer U$1LS.29
- net GPIO_25: now also U$4LS.30; no longer U$1LS.30
- net GPIO_69: now also U$4LS.26; no longer U$1LS.26
- net HSIC_DATA: now also U$4HS.59; no longer U$1HS.59
- net HSIC_STR: now also U$4HS.57; no longer U$1HS.57
- net I2C0_SCL: now also JP2.2, U$4LS.15; no longer JP7.2, U$1LS.15
- net I2C0_SDA: now also JP2.1, U$4LS.17; no longer JP7.1, U$1LS.17
- net I2C1_SCL: now also JP100.2, JP3.4, JP4.2, U$4LS.19; no longer JP1.4, JP2.2, JP5.2, U$1LS.19
- net I2C1_SDA: now also JP100.4, JP3.5, JP4.1, U$4LS.21; no longer JP1.5, JP2.1, JP5.4, U$1LS.21
- net I2C3_SCL: now also U$4HS.36; no longer U$1HS.36
- net I2C3_SDA: now also U$4HS.38; no longer U$1HS.38
- net MCLK0: now also U$4HS.15; no longer U$1HS.15
- net MCLK1: now also U$4HS.17; no longer U$1HS.17
- net N$1: now also JP5.2, U$1.PS; no longer JP3.2, U$2.PS
- net N$10: now also U$2.ECL; no longer U$3.ECL
- net N$11: now also C12.1, R1.2, U$3.OSCO; no longer C25.1, R3.2, U$4.OSCO
- net N$12: now also U$2.INT; no longer U$3.INT
- net N$14: now also IC1.DO, R2.1; no longer IC2.DO, R5.1
- net N$17: now also R4.2, R5.1, U$3.RESET; no longer R1.1, R2.2, U$4.RESET
- net N$2: now also JP4.3, U$1.SDA; no longer JP2.3, U$2.SDA
- net N$3: now also JP4.4, U$1.SCL; no longer JP2.4, U$2.SCL
- net N$4: now also JP1.4, JP100.1; no longer JP4.4, JP5.1
- net N$5: now also JP1.3, JP100.3; no longer JP4.3, JP5.3
- net N$6: now also C21.1, R3.2, U$3.REF; no longer C30.1, R4.2, U$4.REF
- net N$7: now also C11.1, R1.1, U$3.OSIC; no longer C26.1, R3.1, U$4.OSIC
- net N$8: now also U$2.ECA; no longer U$3.ECA
- net N$9: now also U$4A.15; no longer U$1A.15
- net ON: now also U$4LS.4; no longer U$1LS.4
- net RESET0: now also U$4LS.31; no longer U$1LS.31
- net RESET1: now also U$4LS.33; no longer U$1LS.33
- net RESIN: now also U$4LS.6; no longer U$1LS.6
- net SBUS: now also JP11.3; no longer JP8.3
- net SPI0_CLK: now also U$4LS.8; no longer U$1LS.8
- net SPI0_CS_N: now also U$4LS.12; no longer U$1LS.12
- net SPI0_MISO: now also U$4LS.10; no longer U$1LS.10
- net SPI0_MOSI: now also U$4LS.14; no longer U$1LS.14
- net SPI1_CLK: now also U$4HS.9; no longer U$1HS.9
- net SPI1_CS: now also U$4HS.7; no longer U$1HS.7
- net SPI1_MISO: now also U$4HS.11; no longer U$1HS.11
- net SPI1_MOSI: now also U$4HS.1; no longer U$1HS.1
- net SPI_A_CLK: now also U$2.SCL; no longer U$3.SCL
- net SPI_A_CS: now also U$2.NCS; no longer U$3.NCS
- net SPI_A_MISO: now also U$2.AD0; no longer U$3.AD0
- net SPI_A_MOSI: now also U$2.SDA; no longer U$3.SDA
- net SPI_B_CLK: now also JP4.6; no longer JP2.6
- net SPI_B_CS: now also U$1.CSB; no longer U$2.CSB
- net SPI_B_MISO: now also U$1.SDO; no longer U$2.SDO
- net SPI_B_MOSI: now also JP4.5; no longer JP2.5
- net SPKR_OUT_M: now also U$4A.2; no longer U$1A.2
- net SPKR_OUT_P: now also U$4A.1; no longer U$1A.1
- net STANDBY0: now also U$4LS.32; no longer U$1LS.32
- net STANDBY1: now also U$4LS.34; no longer U$1LS.34
- net SYS_DCIN: now also C1.1, C100.1, C33.1, C7.1, U$4LS.36, U$4LS.38; no longer C16.1, C17.1, C8.1, C9.1, U$1LS.36, U$1LS.38
- net UART0_CTS: now also U$4LS.3; no longer U$1LS.3
- net UART0_RX: now also U$4LS.7; no longer U$1LS.7
- net UART0_TX: now also U$4LS.5; no longer U$1LS.5
- net UART1_RX: now also U$4LS.13; no longer U$1LS.13
- net UART1_TX: now also U$4LS.11; no longer U$1LS.11
- net UART_RTS: now also U$4LS.9; no longer U$1LS.9
- net USB_D+: now also JP7.3, U$3.DP, U$4HS.51; no longer JP9.3, U$1HS.51, U$4.DP
- net USB_D-: now also JP7.2, U$3.DM, U$4HS.53; no longer JP9.2, U$1HS.53, U$4.DM
- net VCORE: now also C15.1, C17.1, C26.1, C27.1, U$3.VCORE, U$3.VREGOUT; no longer C106.1, C107.1, C28.1, C29.1, U$4.VCORE, U$4.VREGOUT
- net VDDIO: now also JP3.1; no longer JP1.1
- net VPHY: now also C19.1, C20.1, L1.2, U$3.VPHY; no longer C104.1, C105.1, L2.2, U$4.VPHY
- net VPH_PWR: now also U$4A.3; no longer U$1A.3
- net VPLL: now also C24.1, C25.1, L2.2, U$3.VPLL; no longer C102.1, C103.1, L1.2, U$4.VPLL

Commit message: Fixed more of Josh's fuck ups.
Connections:
- removed net GND_CFILT: U$4A.5
- net GND: now also U$4A.5
Changed lines of the file:
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@@
 <part name="U$4" library="DragonBoard" deviceset="DRAGON-BOARD-TH" device=""/>
 <part name="GND21" library="interface_board-rev13" deviceset="GND" device=""/>
+<part name="GND2" library="interface_board-rev13" deviceset="GND" device=""/>
 </parts>
 <sheets>
@@
 <instance part="GND20" gate="1" x="106.68" y="167.64"/>
 <instance part="U$4" gate="A" x="40.64" y="187.96"/>
+<instance part="GND2" gate="1" x="7.62" y="177.8"/>
 </instances>
 <busses>
@@
 <label x="25.4" y="195.58" size="1.27" layer="95" rot="R180" xref="yes"/>
 <pinref part="U$4" gate="A" pin="3"/>
-</segment>
-</net>
-<net name="GND_CFILT" class="0">
-<segment>
-<wire x1="30.48" y1="193.04" x2="25.4" y2="193.04" width="0.1524" layer="91"/>
-<label x="25.4" y="193.04" size="1.27" layer="95" rot="R180" xref="yes"/>
-<pinref part="U$4" gate="A" pin="5"/>
 </segment>
 </net>
@@
 <junction x="106.68" y="172.72"/>
 </segment>
-</net>
+<segment>
+<pinref part="U$4" gate="A" pin="5"/>
+<wire x1="30.48" y1="193.04" x2="7.62" y2="193.04" width="0.1524" layer="91"/>
+<wire x1="7.62" y1="193.04" x2="7.62" y2="180.34" width="0.1524" layer="91"/>
+<pinref part="GND2" gate="1" pin="GND"/>
+</segment>
+</net>
